Commit message: urdf corregido

File: src/Brazo robotico/urdf2/urdf/urdf2.urdf (robot description, URDF)
Before this commit: robot ROBOT_URDF, 5 links, 4 joints
Links:
- removed link Link_2
- removed link base
- removed link link_5
- added link Link_1, mass 0.235997319223989; collision mesh filename=package://urdf2/meshes/Link_1.STL; visual mesh filename=package://urdf2/meshes/Link_1.STL
- added link eslabon_0, mass 0.89153; collision mesh filename=package://urdf2/meshes/eslabon_0.STL; visual mesh filename=package://urdf2/meshes/eslabon_0.STL
- added link link_2, mass 0.35706117343289; collision mesh filename=package://urdf2/meshes/link_2.STL; visual mesh filename=package://urdf2/meshes/link_2.STL
- link link_3: mass 0.3642 -> 0.197506281990069; geometry collision mesh filename=package://urdf2/meshes/link_3.STL; visual mesh filename=package://urdf2/meshes/link_3.STL
- link link_4: mass 0.20146 -> 0.0567373643332565; geometry collision mesh filename=package://urdf2/meshes/link_4.STL; visual mesh filename=package://urdf2/meshes/link_4.STL
Joints:
- removed joint joint_3
- removed joint joint_4
- removed joint joint_5
- added joint Joint_1: type revolute, parent eslabon_0, child Link_1, origin xyz=0 0 0.145 rpy=0 0 -1.2171, axis 0 0 1, limit lower=0 upper=3.142 effort=300 velocity=3
- added joint Joint_3: type revolute, parent link_2, child link_3, origin xyz=0.06605 0 0.13468 rpy=1.5708 -1.1148 0, axis 0 0 -1, limit lower=0 upper=3.142 effort=200 velocity=3
- added joint Joint_4: type continuous, parent link_3, child link_4, origin xyz=-0.02966 -0.12143 0 rpy=0 0 -1.005, axis 0 0 -1, limit upper=-3.142 effort=200 velocity=3
- joint Joint_2: axis 0 0 1 -> 0 1 0; child Link_2 -> link_2; limit lower=0 upper=3.142 effort=300 velocity=3 -> lower=-1.57 upper=1.57 effort=200 velocity=3; origin xyz=0 0 0.145 rpy=0 0 -0.73283 -> xyz=0 0 0 rpy=0 0 0; parent base -> Link_1; type revolute -> continuous
