Commit message: correcion de commit (?)

File: src/muevelo/config/gazebo_urdf2.urdf (robot description, URDF)
Before this commit: robot urdf2, 6 links, 5 joints
Joints:
- joint Joint_1: limit lower=0 upper=3.142 effort=300 velocity=3 -> lower=0 upper=3.142 effort=30 velocity=3
- joint Joint_2: limit lower=-2 upper=0.3 effort=200 velocity=3 -> lower=-2 upper=0.3 effort=20 velocity=3
- joint Joint_3: limit lower=-1 upper=0.5 effort=200 velocity=3 -> lower=-1 upper=0.5 effort=20 velocity=3
- joint Joint_4: limit effort=200 velocity=3 -> effort=20 velocity=3
